File: photodiode_pcb/photodiode_pcb.sch (KiCad schematic (older format))
At the start: 9 parts, among them J1 Conn_Coaxial

Commit message: old update. Not sure what it contains
Parts:
- removed D3: Photodiode_can, Package_TO_SOT_THT:TO-46-3_Window, symbol my_library:Photodiode_can
- added D3: D_Photo, symbol Device:D_Photo
Connections:
- net GND: now also D3.2 (A)
- net at D1.1 (K), D2.2 (A), R1.2: now also D3.1 (K)
Changed lines of the file:
@@
 $EndDescr
-$Comp
-L my_library:Photodiode_can D3
-U 1 1 5F99588E
-P 4600 3450
-F 0 "D3" V 4504 3608 50  0000 L CNN
-F 1 "Photodiode_can" V 4595 3608 50  0000 L CNN
-F 2 "Package_TO_SOT_THT:TO-46-3_Window" H 4550 3450 50  0001 C CNN
-F 3 "~" H 4550 3450 50  0001 C CNN
-	1    4600 3450
-	0    1    1    0
-$EndComp
 $Comp
 L pspice:DIODE D1
@@
 Wire Wire Line
 	4600 3900 4600 3550
-$Comp
-L power:GND #PWR02
-U 1 1 5F99826F
-P 4400 3650
-F 0 "#PWR02" H 4400 3400 50  0001 C CNN
-F 1 "GND" H 4405 3477 50  0000 C CNN
-F 2 "" H 4400 3650 50  0001 C CNN
-F 3 "" H 4400 3650 50  0001 C CNN
-	1    4400 3650
-	1    0    0    -1
-$EndComp
-Wire Wire Line
-	4400 3650 4400 3500
 Wire Wire Line
 	4600 3250 4600 3150
@@
 $EndComp
 $Comp
-L power:GND #PWR?
+L power:GND #PWR0101
 U 1 1 5F9A91E0
 P 2950 4800
-F 0 "#PWR?" H 2950 4550 50  0001 C CNN
+F 0 "#PWR0101" H 2950 4550 50  0001 C CNN
 F 1 "GND" H 2955 4627 50  0000 C CNN
 F 2 "" H 2950 4800 50  0001 C CNN
@@
 $EndComp
 $Comp
-L power:GND #PWR?
+L power:GND #PWR0102
 U 1 1 5F9A97C4
 P 2950 5200
-F 0 "#PWR?" H 2950 4950 50  0001 C CNN
+F 0 "#PWR0102" H 2950 4950 50  0001 C CNN
 F 1 "GND" H 2955 5027 50  0000 C CNN
 F 2 "" H 2950 5200 50  0001 C CNN
@@
 $EndComp
 $Comp
-L power:GND #PWR?
+L power:GND #PWR0103
 U 1 1 5F9A9B50
 P 2950 5900
-F 0 "#PWR?" H 2950 5650 50  0001 C CNN
+F 0 "#PWR0103" H 2950 5650 50  0001 C CNN
 F 1 "GND" H 2955 5727 50  0000 C CNN
 F 2 "" H 2950 5900 50  0001 C CNN
@@
 $EndComp
 $Comp
-L power:GND #PWR?
+L power:GND #PWR0104
 U 1 1 5F9AA190
 P 2950 5600
-F 0 "#PWR?" H 2950 5350 50  0001 C CNN
+F 0 "#PWR0104" H 2950 5350 50  0001 C CNN
 F 1 "GND" H 2955 5427 50  0000 C CNN
 F 2 "" H 2950 5600 50  0001 C CNN
@@
 	1    0    0    -1
 $EndComp
+$Comp
+L Device:D_Photo D3
+U 1 1 5FF793C0
+P 4600 3450
+F 0 "D3" V 4504 3608 50  0000 L CNN
+F 1 "D_Photo" V 4595 3608 50  0000 L CNN
+F 2 "" H 4550 3450 50  0001 C CNN
+F 3 "~" H 4550 3450 50  0001 C CNN
+	1    4600 3450
+	0    1    1    0
+$EndComp
 $EndSCHEMATC
